File: KiCAD/AmigaPCI-LBC040-REV60/AmigaPCI 68040.kicad_sch (KiCad schematic)
At the start: 0 parts

Commit message: AmigaPCI Local Bus Card Revision 6.0
Other:
- note added: "DESIGNED WITH KICAD 8"
Changed lines of the file:
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@@
 	(title_block
 		(title "AmigaPCI 68040 Local Bus Card")
-		(date "2025-06-29")
-		(rev "5.0")
+		(date "2026-04-07")
+		(rev "6.0")
+	)
+	(text "DESIGNED WITH KICAD 8"
+		(exclude_from_sim no)
+		(at 30.48 196.088 0)
+		(effects
+			(font
+				(size 1.27 1.27)
+			)
+		)
 	)
 	(text "AmigaPCI CPU LOCAL BUS CARD\nMC68040 + 128MB FAAAST RAM\n\n\"THE BRAIN\""
