File: KiCAD/AmigaPCI-LBC040-REV60/CPU.kicad_sch (KiCad schematic)
At the start: 25 parts, among them J100 SNOOP, J101 MMU/CACHE, U200 MC68040, U203 74LVC245

Commit message: AmigaPCI Local Bus Card Revision 6.0
Parts:
- added C139: 0.1uF, Capacitor_SMD:C_0603_1608Metric, symbol Device:C_Small
- added R104, R111: 22R, Resistor_SMD:R_0603_1608Metric, symbol Device:R
- added U112: 74LVC244, Package_SO:TSSOP-20_4.4x6.5mm_P0.65mm, symbol 74xx:74LS244
Connections:
- net _BG-3V is gone; now on net R_W-3V: U203.4 (A2)
- net +3V3: now also C139.2, U112.20 (VCC)
- net GND: now also C139.1, U112.10 (GND), U112.11 (I0b), U112.2 (I0a); no longer U200.172 (_AVEC)
- net R_W: now also R111.1; no longer U200.112 (R_W), U203.15 (B3)
- net R_W-3V: no longer U203.5 (A3)
- net _BB: now also U203.14 (B4); no longer U203.13 (B5)
- net _BB-3V: now also U203.6 (A4); no longer U203.7 (A5)
- net _BG: no longer U203.16 (B2)
- net _MI: now also U203.13 (B5)
- net _TS-3V: now also U203.5 (A3); no longer U203.6 (A4)
- net _TS-CPU: now also U203.15 (B3); no longer U203.14 (B4)
- new net: R104.2, U112.16 (O1a), U112.7 (O1b)
- new net R_W-CPU: R111.2, U200.112 (R_W), U203.16 (B2)
- new net SCLK: U112.17 (I3b), U112.8 (I3a)
- new net SDI: U112.15 (I2b), U112.6 (I2a)
- new net SDO: R104.1
- new net U109_SCK: U112.12 (O3a)
- new net U109_SDI: U112.14 (O2a)
- new net U109_SDO: U112.4 (I1a)
- new net U109_SS: U112.18 (O0a)
- new net U409_SCK: U112.3 (O3b)
- new net U409_SDI: U112.5 (O2b)
- new net U409_SDO: U112.13 (I1b)
- new net U409_SS: U112.9 (O0b)
- new net _AUTOVECTOR: U200.172 (_AVEC)
- new net _MI-3V: U203.7 (A5)
- new net _SPIAEN: U112.19 (OEb)
- new net _SPIBEN: U112.1 (OEa)
Other:
- note added: "FPGA PROGRAM"
