File: KiCAD/AmigaPCI-LBC040-REV60/CardConnector.kicad_sch (KiCad schematic)
At the start: 43 parts, among them CN100 DIN41612_03x40, CN111 SPI, U111 ICE40HX4K-TQ144, U409F2 W25X20CLSN, X100 40MHz

Commit message: AmigaPCI Local Bus Card Revision 6.0
Parts:
- removed CN100: DIN41612_03x40, AmigaPCI:DIN41612_R_3x40_Male_Vertical_THT, symbol AmigaPCI-Symbols:DIN41612_03x40
- removed R111: 22R, Resistor_SMD:R_0603_1608Metric, symbol Device:R
- added CN100: DIN41612_03x50, AmigaPCI:DIN41612_C_3x50_Male_Vertical_THT, symbol AmigaPCI-Symbols:DIN41612_03x50
- X100: value 40MHz -> 80MHz
Connections:
- net _BG-3V is gone; now on net _BG: U111.96 (IO1_146)
- net +1V2: now also CN100.a13 (Pin_a13)
- net +3V3: now also CN100.a28 (Pin_a28), CN100.a41 (Pin_a41), CN100.a48 (Pin_a48), CN100.a49 (Pin_a49), CN100.b12 (Pin_b12), CN100.b13 (Pin_b13), CN100.c20 (Pin_c20), CN100.c3 (Pin_c3), CN100.c7 (Pin_c7)
- net +3V3SB: now also CN100.c21 (Pin_c21)
- net +5V: now also CN100.a1 (Pin_a1), CN100.a14 (Pin_a14), CN100.a29 (Pin_a29), CN100.a32 (Pin_a32), CN100.a33 (Pin_a33), CN100.a40 (Pin_a40), CN100.a50 (Pin_a50), CN100.c12 (Pin_c12), CN100.c6 (Pin_c6)
- net A0: now also CN100.b10 (Pin_b10)
- net A10: now also CN100.b17 (Pin_b17)
- net A11: now also CN100.a17 (Pin_a17)
- net A12: now also CN100.a9 (Pin_a9)
- net A13: now also CN100.b9 (Pin_b9)
- net A14: now also CN100.a10 (Pin_a10)
- net A15: now also CN100.c10 (Pin_c10)
- net A16: now also CN100.c47 (Pin_c47)
- net A17: now also CN100.b47 (Pin_b47)
- net A18: now also CN100.a47 (Pin_a47)
- net A19: now also CN100.c46 (Pin_c46)
- net A2: now also CN100.b11 (Pin_b11)
- net A20: now also CN100.b46 (Pin_b46)
- net A21: now also CN100.c45 (Pin_c45)
- net A22: now also CN100.a42 (Pin_a42)
- net A23: now also CN100.a46 (Pin_a46)
- net A24: now also CN100.a43 (Pin_a43)
- net A25: now also CN100.b45 (Pin_b45)
- net A26: now also CN100.b42 (Pin_b42)
- net A27: now also CN100.c44 (Pin_c44)
- net A28: now also CN100.c42 (Pin_c42)
- net A29: now also CN100.c43 (Pin_c43)
- net A3: now also CN100.c11 (Pin_c11)
- net A30: now also CN100.b43 (Pin_b43)
- net A31: now also CN100.b44 (Pin_b44)
- net A4: now also CN100.a12 (Pin_a12)
- net A5: now also CN100.b15 (Pin_b15)
- net A6: now also CN100.a15 (Pin_a15)
- net A7: now also CN100.b16 (Pin_b16)
- net A8: now also CN100.a16 (Pin_a16)
- net A9: now also CN100.c15 (Pin_c15)
- net AA1: now also CN100.a11 (Pin_a11)
- net BCLKC: now also CN100.a35 (Pin_a35)
- net BUFDIR: now also U111.135 (IO0_213); no longer U111.136 (IO0_214)
- net CDONE: now also CN100.b29 (Pin_b29)
- net DA0: now also CN100.a39 (Pin_a39)
- net DA1: now also CN100.c38 (Pin_c38)
- net DA10: now also CN100.c33 (Pin_c33)
- net DA11: now also CN100.b33 (Pin_b33)
- net DA12: now also CN100.c32 (Pin_c32)
- net DA13: now also CN100.c31 (Pin_c31)
- net DA14: now also CN100.c27 (Pin_c27)
- net DA15: now also CN100.b27 (Pin_b27)
- net DA16: now also CN100.b32 (Pin_b32)
- net DA17: now also CN100.a27 (Pin_a27)
- net DA18: now also CN100.b31 (Pin_b31)
- net DA19: now also CN100.b26 (Pin_b26)
- net DA2: now also CN100.a38 (Pin_a38)
- net DA20: now also CN100.a25 (Pin_a25)
- net DA21: now also CN100.c22 (Pin_c22)
- net DA22: now also CN100.b25 (Pin_b25)
- net DA23: now also CN100.c26 (Pin_c26)
- net DA24: now also CN100.b21 (Pin_b21)
- net DA25: now also CN100.a26 (Pin_a26)
- net DA26: now also CN100.a21 (Pin_a21)
- net DA27: now also CN100.b23 (Pin_b23)
- net DA28: now also CN100.b20 (Pin_b20)
- net DA29: now also CN100.a23 (Pin_a23)
- net DA3: now also CN100.b39 (Pin_b39)
- net DA30: now also CN100.b22 (Pin_b22)
- net DA31: now also CN100.a22 (Pin_a22)
- net DA4: now also CN100.b38 (Pin_b38)
- net DA5: now also CN100.c37 (Pin_c37)
- net DA6: now also CN100.b37 (Pin_b37)
- net DA7: now also CN100.c36 (Pin_c36)
- net DA8: now also CN100.a34 (Pin_a34)
- net DA9: now also CN100.b34 (Pin_b34)
- net GND: now also CN100.a2 (Pin_a2), CN100.a31 (Pin_a31), CN100.a36 (Pin_a36), CN100.a37 (Pin_a37), CN100.a44 (Pin_a44), CN100.a45 (Pin_a45), CN100.b14 (Pin_b14), CN100.b6 (Pin_b6), CN100.c16 (Pin_c16), CN100.c17 (Pin_c17), CN100.c24 (Pin_c24), CN100.c25 (Pin_c25), CN100.c4 (Pin_c4), CN100.c49 (Pin_c49), CN100.c50 (Pin_c50), CN100.c8 (Pin_c8), CN100.c9 (Pin_c9)
- net PORTSIZE: now also CN100.a8 (Pin_a8)
- net R_W: now also CN100.b19 (Pin_b19)
- net SCL: now also CN100.c40 (Pin_c40)
- net SDA: now also CN100.b41 (Pin_b41)
- net TM0: now also CN100.a19 (Pin_a19)
- net TM1: now also CN100.c19 (Pin_c19)
- net TM2: now also CN100.a20 (Pin_a20)
- net TT0: now also CN100.c39 (Pin_c39)
- net TT1: now also CN100.b40 (Pin_b40)
- net _BB: now also CN100.b8 (Pin_b8)
- net _BG: now also CN100.c29 (Pin_c29)
- net _BR: now also CN100.a18 (Pin_a18)
- net _BUFEN: now also U111.136 (IO0_214); no longer U111.135 (IO0_213)
- net _CPURST: now also CN100.c18 (Pin_c18)
- net _INT2: now also CN100.c13 (Pin_c13)
- net _INT6: now also CN100.b30 (Pin_b30)
- net _IPL0: now also CN100.c34 (Pin_c34)
- net _IPL1: now also CN100.c35 (Pin_c35)
- net _IPL2: now also CN100.b36 (Pin_b36)
- net _LBEN: now also U111.60 (IO2_95), CN100.a4 (Pin_a4); no longer U111.48 (IO2_80)
- net _LOCK: now also CN100.b18 (Pin_b18)
- net _RESET: now also CN100.b35 (Pin_b35)
- net _RSTOUT: now also CN100.c41 (Pin_c41)
- net _TACK: now also CN100.b28 (Pin_b28)
- net _TBI: now also U111.48 (IO2_80), CN100.a30 (Pin_a30); no longer U111.55 (IO2_91)
- net _TCI: now also CN100.c30 (Pin_c30)
- net _TEA: now also CN100.c28 (Pin_c28)
- net _TS: now also CN100.b24 (Pin_b24)
- net _TS-3V: now also U111.20 (IO3_13B_GBIN7); no longer U111.125 (IO0_192)
- net at R115.1: now also U111.55 (IO2_91); no longer U111.49 (IO2_81_GBIN5)
- net at R119.1: now also CN100.c23 (Pin_c23)
- net _TS-RAM: now reaches U111.39 (IO2_61)
- net at U111.52 (IO2_82_GBIN4): no longer R116.1
- net at U111.61 (IO2_96): now also R116.1
- net at R120.1: now also CN100.a24 (Pin_a24)
- net CLK40 renamed CLKCPU
- new net LBC: CN100.c14 (Pin_c14)
- new net SCLK: CN100.a5 (Pin_a5)
- new net SDI: CN100.c5 (Pin_c5)
- new net SDO: CN100.b5 (Pin_b5)
- new net _AUTOVECTOR: CN100.b1 (Pin_b1)
- new net _DATARDY: CN100.b3 (Pin_b3)
- new net _SPIAEN: CN100.a3 (Pin_a3)
- new net _SPIBEN: CN100.c2 (Pin_c2)
- no-connect marks 8 -> 17
Other:
- moved on the sheet: C113, C114, C115, C116, C117, C135, C138, H1, H2, R113, R115, R116
