File: KiCAD/AmigaPCI-LBC040-REV60/FastMem.kicad_sch (KiCad schematic)
At the start: 36 parts, among them CN400 SPI, J1 _CS0, J2 _CS1, J3 _RAS, J4 _CAS, J5 _WE, J6 CLKEN, J7 RAMCLK, U400 ICE40HX1K-VQ100, U400F1 W25X20CLSN, U401 SDRAM(16Mx32), U402 SDRAM(16Mx32)

Commit message: AmigaPCI Local Bus Card Revision 6.0
Connections:
- net _TS-3V is gone; now on net SIZ1-3V: U400.57 (IOR_57)
- net BCLKB: now also U400.63 (IOR_61_GBIN2); no longer U400.53 (IOR_54)
- net LVA22: now also U400.27 (IOB_27); no longer U400.28 (IOB_28)
- net LVA25: now also U400.30 (IOB_30); no longer U400.34 (IOB_36_GBIN4)
- net LVA26: now also U400.28 (IOB_28); no longer U400.29 (IOB_29)
- net LVA28: now also U400.29 (IOB_29); no longer U400.30 (IOB_30)
- net LVA30: now also U400.41 (IOB_42_CBSEL0); no longer U400.33 (IOB_35_GBIN5)
- net LVA31: now also U400.42 (IOB_43_CBSEL1); no longer U400.27 (IOB_27)
- net RAMCLKB: now also U400.90 (IOT_85_GBIN0); no longer U400.52 (IOR_53)
- net SIZ0-3V: now also U400.59 (IOR_58); no longer U400.60 (IOR_59)
- net SIZ1-3V: no longer U400.59 (IOR_58)
- net _EM1CS: now also U400.60 (IOR_59); no longer U400.90 (IOT_85_GBIN0)
- net _LBEN: now also U400.53 (IOR_54); no longer U400.54 (IOR_55)
- net _LLBE: now also U400.33 (IOB_35_GBIN5); no longer U400.42 (IOB_43_CBSEL1)
- net _LMBE: now also U400.34 (IOB_36_GBIN4); no longer U400.41 (IOB_42_CBSEL0)
- net _RESET: now also U400.52 (IOR_53); no longer U400.63 (IOR_61_GBIN2)
- net _TA-CPU: now also U400.54 (IOR_55); no longer U400.56 (IOR_56)
- net _DATARDY: now reaches U400.2 (IOL_1B)
- net _MI renamed _TS-RAM
- new net _MI-3V: U400.56 (IOR_56)
- no-connect marks 2 -> 1
