File: KiCAD/AmigaPCI-LBC040-REV60/FastMem.kicad_sch (KiCad schematic)
At the start: 36 parts, among them CN400 SPI, J1 _CS0, J2 _CS1, J3 _RAS, J4 _CAS, J5 _WE, J6 CLKEN, J7 RAMCLK, U400 ICE40HX1K-VQ100, U400F1 W25X20CLSN, U401 SDRAM(16Mx32), U402 SDRAM(16Mx32)

Commit message: Add JLCPCB part numbers to KiCAD schematic.
Parts:
- C400, C401, C402, C403, C404, C405, C406, C407, C408, C409, C410, C411, C412, C413, C414, C415, C416, C417, C418, C422, C423, C425: LCSC (none) -> C14663
- CN400: LCSC (none) -> C37208
- R400, R401: LCSC (none) -> C25804
- U400: LCSC (none) -> C1519043
- U400F1: LCSC (none) -> C34591
- U401, U402: LCSC (none) -> C17489827
