File: KiCAD/AmigaPCI-LBC040-REV60/level_shift.kicad_sch (KiCad schematic)
At the start: 30 parts, among them U101 74LVC245, U102 74LVC245, U103 74LVC245, U104 74LVC245, U105 74LVC245, U106 74LVC245, U107 74LVC245, U108 74LVC245, U109 SN74LVC16T245DLR, U110 SN74LVC16T245DLR, U113 74LVC1G125, U115 74LVC1G125

Commit message: AmigaPCI Local Bus Card Revision 6.0
Parts:
- removed C118, C119, C120, C121: 0.1uF, Capacitor_SMD:C_0603_1608Metric, symbol Device:C_Small
- removed U109, U110: SN74LVC16T245DLR, AmigaPCI:48-BSSOP, symbol AmigaPCI-Symbols:SN74LVC16T245DLR
- added U109, U110, U116, U117: 74LVC245, Package_SO:TSSOP-20_4.4x6.5mm_P0.65mm, symbol AmigaPCI-Symbols:74LVC245
Connections:
- net +3V3: now also U109.20 (VCC), U110.20 (VCC), U116.20 (VCC), U117.20 (VCC)
- net BUFDIR: now also U109.1 (A->B), U110.1 (A->B), U116.1 (A->B), U117.1 (A->B)
- net DA0: now also U109.9 (A7)
- net DA1: now also U109.5 (A3)
- net DA10: now also U110.6 (A4)
- net DA11: now also U110.7 (A5)
- net DA12: now also U110.4 (A2)
- net DA13: now also U110.2 (A0)
- net DA14: now also U116.7 (A5)
- net DA15: now also U116.8 (A6)
- net DA16: now also U110.5 (A3)
- net DA17: now also U116.9 (A7)
- net DA18: now also U110.3 (A1)
- net DA19: now also U116.5 (A3)
- net DA2: now also U109.7 (A5)
- net DA20: now also U116.3 (A1)
- net DA21: now also U117.5 (A3)
- net DA22: now also U116.2 (A0)
- net DA23: now also U116.4 (A2)
- net DA24: now also U117.3 (A1)
- net DA25: now also U116.6 (A4)
- net DA26: now also U117.4 (A2)
- net DA27: now also U117.8 (A6)
- net DA28: now also U117.2 (A0)
- net DA29: now also U117.9 (A7)
- net DA3: now also U109.8 (A6)
- net DA30: now also U117.6 (A4)
- net DA31: now also U117.7 (A5)
- net DA4: now also U109.6 (A4)
- net DA5: now also U109.3 (A1)
- net DA6: now also U109.4 (A2)
- net DA7: now also U109.2 (A0)
- net DA8: now also U110.9 (A7)
- net DA9: now also U110.8 (A6)
- net GND: now also U109.10 (GND), U110.10 (GND), U116.10 (GND), U117.10 (GND)
- net LVDB0: now also U109.11 (B7)
- net LVDB1: now also U109.15 (B3)
- net LVDB10: now also U110.14 (B4)
- net LVDB11: now also U110.13 (B5)
- net LVDB12: now also U110.16 (B2)
- net LVDB13: now also U110.18 (B0)
- net LVDB14: now also U116.13 (B5)
- net LVDB15: now also U116.12 (B6)
- net LVDB16: now also U110.15 (B3)
- net LVDB17: now also U116.11 (B7)
- net LVDB18: now also U110.17 (B1)
- net LVDB19: now also U116.15 (B3)
- net LVDB2: now also U109.13 (B5)
- net LVDB20: now also U116.17 (B1)
- net LVDB21: now also U117.15 (B3)
- net LVDB22: now also U116.18 (B0)
- net LVDB23: now also U116.16 (B2)
- net LVDB24: now also U117.17 (B1)
- net LVDB25: now also U116.14 (B4)
- net LVDB26: now also U117.16 (B2)
- net LVDB27: now also U117.12 (B6)
- net LVDB28: now also U117.18 (B0)
- net LVDB29: now also U117.11 (B7)
- net LVDB3: now also U109.12 (B6)
- net LVDB30: now also U117.14 (B4)
- net LVDB31: now also U117.13 (B5)
- net LVDB4: now also U109.14 (B4)
- net LVDB5: now also U109.17 (B1)
- net LVDB6: now also U109.16 (B2)
- net LVDB7: now also U109.18 (B0)
- net LVDB8: now also U110.11 (B7)
- net LVDB9: now also U110.12 (B6)
- net _BUFEN: now also U109.19 (CE), U110.19 (CE), U116.19 (CE), U117.19 (CE)
Other:
- moved on the sheet: C109, C110, C111, C112
