File: KiCAD/AmigaPCI-LBC040-REV60/level_shift.kicad_sch (KiCad schematic)
At the start: 28 parts, among them U101 74LVC245, U102 74LVC245, U103 74LVC245, U104 74LVC245, U105 74LVC245, U106 74LVC245, U107 74LVC245, U108 74LVC245, U109 74LVC245, U110 74LVC245, U113 74LVC1G125, U115 74LVC1G125, U116 74LVC245, U117 74LVC245

Commit message: Add JLCPCB part numbers to KiCAD schematic.
Parts:
- C101, C102, C103, C104, C105, C106, C107, C108, C109, C110, C111, C112, C140, C142: LCSC (none) -> C14663
- U101, U102, U103, U104, U105, U106, U107, U108, U109, U110, U116, U117: LCSC (none) -> C7848
- U113, U115: LCSC (none) -> C151022
